File: BatteryPack/BatteryPack.kicad_pcb (KiCad board)
At the start: 2 copper layers, 40.8 x 22.9 mm, 27 parts, among them Q1 IRFR220NTRPBF, Q2 BC817-40, U2 ETA3000S2G, U3 ETA3000S2G, U4 ETA3000S2G

Commit message: Add files via upload
Parts:
- removed Q1: IRFR220NTRPBF, Package_TO_SOT_SMD:TO-252-2
- removed Q2: BC817-40, Package_TO_SOT_SMD:SOT-23
- removed R7, R9: 1R2, Resistor_SMD:R_1206_3216Metric_Pad1.30x1.75mm_HandSolder
- removed R8: 1k, Resistor_SMD:R_0603_1608Metric_Pad0.98x0.95mm_HandSolder
- added F1: MF-MSMF150/24X-2, Fuse:Fuse_1812_4532Metric_Pad1.30x3.40mm_HandSolder, F.Cu at (122.0, 110.2)
Routing:
- net Net-(Q1-S): track 21.7 -> 0.00 mm
- net Net-(Q1-G): track 16.4 -> 0.00 mm
- net Net-(BT1-+): track 43.3 -> 41.6 mm
- net /pack+: track 24.7 -> 23.5 mm
